Commit message: Changed driver_r1.py to get ros param, README, use launch to run driver_r1.py, Added stl models

File: r1_description/urdf/r1.urdf.xacro (robot description, xacro)
@@ -7,11 +7,11 @@
     <parent link="base_footprint"/>
     <child link="base_link" />
-    <origin xyz="0 0 0.050" rpy="0 0 0.0"/>
+    <origin xyz="0 0.0 0.050" rpy="0 0 0.0"/>
   </joint>
   <link name="base_link">
     <visual>
-      <origin xyz="-0.2 0 0.0" rpy="0 0 0.0"/>
+      <origin xyz="0.1 0.28 0.25" rpy="3.14 0 -1.57"/>
       <geometry>
-        <mesh filename="file://$(arg meshDirectory)bases/waffle_pi_base.stl" scale="0.0025 0.0016 0.0025"/>
+        <mesh filename="file://$(arg meshDirectory)bases/R1_body.stl" scale="0.001 0.001 0.001"/>
       </geometry>
       <material name="light_black"/>
@@ -34,12 +34,12 @@
     <parent link="base_link"/>
     <child link="wheel_left_link"/>
-    <origin xyz="0.0 0.29 0.11" rpy="-1.57 0 0"/>
+    <origin xyz="0.0 0.29 0.10" rpy="1.57 0.0 0"/>
     <axis xyz="0 0 1"/>
   </joint>
   <link name="wheel_left_link">
     <visual>
-      <origin xyz="0 0 0" rpy="0.0 0 0"/>
+      <origin xyz="-0.11 -0.07 0.10" rpy="-1.57 0 0"/>
       <geometry>
-        <mesh filename="file://$(arg meshDirectory)wheels/left_tire.stl" scale="0.0035 0.0035 0.0035"/>
+        <mesh filename="file://$(arg meshDirectory)wheels/wheel.stl" scale="0.001 0.001 0.001"/>
       </geometry>
       <material name="dark"/>
@@ -62,12 +62,12 @@
     <parent link="base_link"/>
     <child link="wheel_right_link"/>
-    <origin xyz="0.0 -0.29 0.11" rpy="-1.57 0 0"/>
+    <origin xyz="0.0 -0.29 0.10" rpy="-1.57 0 0"/>
     <axis xyz="0 0 1"/>
   </joint>
   <link name="wheel_right_link">
     <visual>
-      <origin xyz="0 0 0" rpy="0.0 0 0"/>
+      <origin xyz="-0.11 0.07 -0.122" rpy="1.57 0 0"/>
       <geometry>
-        <mesh filename="file://$(arg meshDirectory)wheels/right_tire.stl" scale="0.0035 0.0035 0.0035"/>
+        <mesh filename="file://$(arg meshDirectory)wheels/wheel.stl" scale="0.001 0.001 0.001"/>
       </geometry>
       <material name="dark"/>
@@ -90,5 +90,5 @@
     <parent link="base_link"/>
     <child link="caster_back_right_link"/>
-    <origin xyz="-0.177 -0.064 -0.004" rpy="-1.57 0 0"/>
+    <origin xyz="-0.38 -0.16 0.06" rpy="-1.57 0 0"/>
   </joint>
   <link name="caster_back_right_link">
@@ -96,5 +96,5 @@
       <origin xyz="0 0.001 0" rpy="0 0 0"/>
       <geometry>
-        <box size="0.030 0.009 0.020"/>
+        <box size="0.040 0.02 0.020"/>
       </geometry>
     </collision>
@@ -110,5 +110,5 @@
     <parent link="base_link"/>
     <child link="caster_back_left_link"/>
-    <origin xyz="-0.177 0.064 -0.004" rpy="-1.57 0 0"/>
+    <origin xyz="-0.38 0.16 0.06" rpy="-1.57 0 0"/>
   </joint>
   <link name="caster_back_left_link">

Commit message: Experimental modification

File: r1_description/urdf/r1.urdf.xacro (robot description, xacro)
@@ -1,13 +1,30 @@
 <?xml version="1.0" ?>
 <robot name="omorobot_r1" xmlns:xacro="http://ros.org/wiki/xacro">
+  <xacro:arg name="meshDirectory" default="$(find omoros)/r1_description/meshes/" />
   <xacro:include filename="$(find omoros)/r1_description/urdf/common_properties.xacro"/>
   <xacro:include filename="$(find omoros)/r1_description/urdf/r1.gazebo.xacro"/>
-  <link name="base_footprint"/>
-  <joint name="base_joint" type="fixed">
-    <parent link="base_footprint"/>
-    <child link="base_link" />
-    <origin xyz="0 0.0 0.050" rpy="0 0 0.0"/>
-  </joint>
+  <link name='odom'/>
   <link name="base_link">
+    <inertial>
+      <origin xyz="0 0 0" rpy="0 0 0"/>
+      <mass value="15.0"/>
+      <inertia ixx="0.1" ixy="0" ixz="0"
+               iyy="0.1" iyz="0"
+               izz="0.1" />
+    </inertial>
+    <collision name='collision'>
+      <origin xyz="0 0 0.036" rpy=" 0 0 0"/>
+      <geometry>
+        <box size=".22 0.08 0.003" />
+      </geometry>
+    </collision>
+    <visual name='base_link_visual'>
+      <origin xyz="0 0 0.036" rpy=" 0 0 0"/>
+      <geometry>
+        <box size="0.22 0.08 0.003"/>
+      </geometry>
+    </visual>
+  </link>
+  <link name="omorobot_r1_body">
     <visual>
       <origin xyz="0.1 0.28 0.25" rpy="3.14 0 -1.57"/>
@@ -17,24 +34,5 @@
       <material name="light_black"/>
     </visual>
-    <collision>
-      <origin xyz="-0.064 0 0.047" rpy="0 0 0"/>
-      <geometry>
-        <box size="0.5 0.5 0.4"/>
-      </geometry>
-    </collision>
-    <inertial>
-      <origin xyz="0 0 0" rpy="0 0 0"/>
-      <mass value="1.3729096e+00"/>
-      <inertia ixx="8.7002718e-03" ixy="-4.7576583e-05" ixz="1.1160499e-04"
-               iyy="8.6195418e-03" iyz="-3.5422299e-06"
-               izz="1.4612727e-02" />
-    </inertial>
   </link>
-  <joint name="wheel_left_joint" type="continuous">
-    <parent link="base_link"/>
-    <child link="wheel_left_link"/>
-    <origin xyz="0.0 0.29 0.10" rpy="1.57 0.0 0"/>
-    <axis xyz="0 0 1"/>
-  </joint>
   <link name="wheel_left_link">
     <visual>
@@ -53,16 +51,10 @@
     <inertial>
       <origin xyz="0 0 0" />
-      <mass value="2.8498940e-02" />
-      <inertia ixx="1.1175580e-05" ixy="-4.2369783e-11" ixz="-5.9381719e-09"
-               iyy="1.1192413e-05" iyz="-1.4400107e-11"
-               izz="2.0712558e-05" />
+      <mass value="2" />
+      <inertia ixx="0.1" ixy="0.0" ixz="0.0"
+               iyy="0.1" iyz="0.0"
+               izz="0.1" />
       </inertial>
   </link>
-  <joint name="wheel_right_joint" type="continuous">
-    <parent link="base_link"/>
-    <child link="wheel_right_link"/>
-    <origin xyz="0.0 -0.29 0.10" rpy="-1.57 0 0"/>
-    <axis xyz="0 0 1"/>
-  </joint>
   <link name="wheel_right_link">
     <visual>
@@ -81,15 +73,10 @@
     <inertial>
       <origin xyz="0 0 0" />
-      <mass value="2.8498940e-02" />
-      <inertia ixx="1.1175580e-05" ixy="-4.2369783e-11" ixz="-5.9381719e-09"
-               iyy="1.1192413e-05" iyz="-1.4400107e-11"
-               izz="2.0712558e-05" />
+      <mass value="2" />
+      <inertia ixx="0.1" ixy="0.0" ixz="0.0"
+               iyy="0.1" iyz="0.0"
+               izz="0.1" />
       </inertial>
   </link>
-  <joint name="caster_back_right_joint" type="fixed">
-    <parent link="base_link"/>
-    <child link="caster_back_right_link"/>
-    <origin xyz="-0.38 -0.16 0.06" rpy="-1.57 0 0"/>
-  </joint>
   <link name="caster_back_right_link">
     <collision>
@@ -107,9 +94,4 @@
     </inertial>
   </link>
-  <joint name="caster_back_left_joint" type="fixed">
-    <parent link="base_link"/>
-    <child link="caster_back_left_link"/>
-    <origin xyz="-0.38 0.16 0.06" rpy="-1.57 0 0"/>
-  </joint>
   <link name="caster_back_left_link">
     <collision>
@@ -127,15 +109,5 @@
     </inertial>
   </link>
-  <joint name="imu_joint" type="fixed">
-    <parent link="base_link"/>
-    <child link="imu_link"/>
-    <origin xyz="0.0 0 0.068" rpy="0 0 0"/>
-  </joint>
   <link name="imu_link"/>
-  <joint name="scan_joint" type="fixed">
-    <parent link="base_link"/>
-    <child link="base_scan"/>
-    <origin xyz="0.0 0 0.5" rpy="0.0 0 0.0"/>
-  </joint>
   <link name="base_scan">
     <visual>
@@ -160,9 +132,4 @@
     </inertial>
   </link>
-  <joint name="camera_joint" type="fixed">
-    <origin xyz="0.073 -0.011 0.084" rpy="0 0 0"/>
-    <parent link="base_link"/>
-    <child link="camera_link"/>
-  </joint>
   <link name="camera_link">
     <collision>
@@ -173,3 +140,51 @@
     </collision>
   </link>
+<!-- Joints -->
+  <joint name="odom_to_base" type="floating">
+    <parent link="odom"/>
+    <child link="base_link"/>
+    <origin xyz="0 0 0.0" rpy="0 0 0"/>
+  </joint>
+  <joint name="wheel_right_joint" type="continuous">
+    <parent link="base_link"/>
+    <child link="wheel_right_link"/>
+    <origin xyz="0.0 -0.29 0.10" rpy="-1.57 0 0"/>
+    <axis xyz="0 0 1"/>
+  </joint>
+  <joint name="wheel_left_joint" type="continuous">
+    <parent link="base_link"/>
+    <child link="wheel_left_link"/>
+    <origin xyz="0.0 0.29 0.10" rpy="1.57 0.0 0"/>
+    <axis xyz="0 0 1"/>
+  </joint>
+  <joint name="caster_back_right_joint" type="fixed">
+    <parent link="base_link"/>
+    <child link="caster_back_right_link"/>
+    <origin xyz="-0.38 -0.16 0.06" rpy="-1.57 0 0"/>
+  </joint>
+  <joint name="caster_back_left_joint" type="fixed">
+    <parent link="base_link"/>
+    <child link="caster_back_left_link"/>
+    <origin xyz="-0.38 0.16 0.06" rpy="-1.57 0 0"/>
+  </joint>
+  <joint name="base_to_body">
+    <origin xyz="0.015 0 0.1" rpy="0 0 0"/>
+    <child link="omorobot_r1_body"/>
+    <parent link="base_link"/>
+  </joint>
+  <joint name="imu_joint" type="fixed">
+    <parent link="base_link"/>
+    <child link="imu_link"/>
+    <origin xyz="0.0 0 0.068" rpy="0 0 0"/>
+  </joint>
+  <joint name="scan_joint" type="fixed">
+    <parent link="base_link"/>
+    <child link="base_scan"/>
+    <origin xyz="0.0 0 0.5" rpy="0.0 0 0.0"/>
+  </joint>
+  <joint name="camera_joint" type="fixed">
+    <origin xyz="0.073 -0.011 0.084" rpy="0 0 0"/>
+    <parent link="base_link"/>
+    <child link="camera_link"/>
+  </joint>
 </robot>
